Commit message: added mobile_base for RVIZ, orientation needs to be changed

File: xarm_description/urdf/xarm6.urdf.xacro (robot description, xacro)
@@ -25,4 +25,41 @@
       <color rgba="0.753 0.753 0.753 1.0"/>
     </material>
+    <xacro:if value="${mobile_base}">
+    <link name="${prefix}mobile_base">
+      <visual>
+        <origin
+          xyz="0 0 0"
+          rpy="0 0 0" />
+        <geometry>
+          <mesh
+            filename="package://xarm_description/meshes/mobile_base/mobile_base_reduced.stl" />
+        </geometry>
+        <material name="Silver" />
+      </visual>
+      <collision>
+        <origin
+          xyz="0 0 0"
+          rpy="0 0 0" />
+        <geometry>
+          <mesh
+            filename="package://xarm_description/meshes/mobile_base/mobile_base_reduced.stl" />
+        </geometry>
+      </collision>
+    </link>
+  </xacro:if>
+  <xacro:unless value="${mobile_base}">
+    <link name="${prefix}mobile_base"/>
+  </xacro:unless>
+  <joint
+    name="${prefix}joint_mobile_base"
+    type="fixed">
+    <origin
+      xyz="0 0 0"
+      rpy="0 0 0" />
+    <parent
+      link="${prefix}mobile_base" />
+    <child
+      link="${prefix}link_base" />
+  </joint>
     <link name="${prefix}link_base">
       <visual>

File: xarm_description/urdf/xarm6_robot.urdf.xacro (robot description, xacro)
@@ -20,4 +20,5 @@
   <!-- <xacro:arg name="add_realsense_d435i" default="false"/> -->
   <xacro:arg name="add_realsense_d435i" default="true"/>
+  <xacro:arg name="add_mobile_base" default="true"/>
   <!-- load xarm6 robot -->
   <xacro:include filename="$(find xarm_description)/urdf/xarm6_robot_macro.xacro" />
@@ -25,4 +26,5 @@
     effort_control="$(arg effort_control)" velocity_control="$(arg velocity_control)"
     rs_d435i="$(arg add_realsense_d435i)"
+    mobile_base="$(arg add_mobile_base)"
     add_other_geometry="$(arg add_other_geometry)"
     geometry_type="$(arg geometry_type)" geometry_mass="$(arg geometry_mass)"

File: xarm_description/urdf/xarm6_robot_macro.xacro (robot description, xacro)
@@ -2,5 +2,5 @@
 <robot xmlns:xacro="http://ros.org/wiki/xacro" name="xarm6" >
   <xacro:macro name="xarm6_robot" params="prefix:='' namespace:='xarm' limited:='false' effort_control:='false'
-    velocity_control:='false' attach_to:='world' xyz:='0 0 0' rpy:='0 0 0' load_gazebo_plugin:='true' rs_d435i:='false'
+    velocity_control:='false' attach_to:='world' xyz:='0 0 0' rpy:='0 0 0' load_gazebo_plugin:='true' rs_d435i:='false' mobile_base='false'
     add_other_geometry:='false'
     geometry_type:='box' geometry_mass:='0.1'
@@ -25,7 +25,12 @@
       <link name="world" />
     </xacro:if>
+    <!-- <joint name="${prefix}world_joint" type="fixed">
+      <parent link="${attach_to}" />
+      <child link = "${prefix}link_base" />
+      <origin xyz="${xyz}" rpy="${rpy}" />
+    </joint> -->
     <joint name="${prefix}world_joint" type="fixed">
       <parent link="${attach_to}" />
-      <child link = "${prefix}link_base" />
+      <child link = "${prefix}mobile_base" />
       <origin xyz="${xyz}" rpy="${rpy}" />
     </joint>
